Commit message: Use package:// mesh paths in the URDF

File: urdf/stretch.urdf (robot description, URDF)
Before this commit: robot stretch_description, 44 links, 43 joints
Links:
- link base_link: geometry collision mesh filename=package://stretch_description/meshes/base_link.STL; visual mesh filename=package://stretch_description/meshes/base_link.STL
- link camera_link: geometry collision box size=0.02505 0.09 0.025; visual mesh filename=package://stretch_description/meshes/d435.dae
- link caster_link: geometry collision sphere radius=0.032; visual mesh filename=package://stretch_description/meshes/omni_wheel_m.STL
- link laser: geometry collision mesh filename=package://stretch_description/meshes/laser.STL; visual mesh filename=package://stretch_description/meshes/laser.STL
- link link_arm_l0: geometry collision mesh filename=package://stretch_description/meshes/link_arm_l0.STL; visual mesh filename=package://stretch_description/meshes/link_arm_l0.STL
- link link_arm_l1: geometry collision mesh filename=package://stretch_description/meshes/link_arm_l1.STL; visual mesh filename=package://stretch_description/meshes/link_arm_l1.STL
- link link_arm_l2: geometry collision mesh filename=package://stretch_description/meshes/link_arm_l2.STL; visual mesh filename=package://stretch_description/meshes/link_arm_l2.STL
- link link_arm_l3: geometry collision mesh filename=package://stretch_description/meshes/link_arm_l3.STL; visual mesh filename=package://stretch_description/meshes/link_arm_l3.STL
- link link_arm_l4: geometry collision mesh filename=package://stretch_description/meshes/link_arm_l4.STL; visual mesh filename=package://stretch_description/meshes/link_arm_l4.STL
- link link_aruco_inner_wrist: geometry collision mesh filename=package://stretch_description/meshes/link_aruco_inner_wrist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; visual mesh filename=package://stretch_description/meshes/link_aruco_inner_wrist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
- link link_aruco_left_base: geometry collision mesh filename=package://stretch_description/meshes/link_aruco_left_base.S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; visual mesh filename=package://stretch_description/meshes/link_aruco_left_base.S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
- link link_aruco_right_base: geometry collision mesh filename=package://stretch_description/meshes/link_aruco_right_base.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; visual mesh filename=package://stretch_description/meshes/link_aruco_right_base.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
- link link_aruco_shoulder: geometry collision mesh filename=package://stretch_description/meshes/link_aruco_shoulder.STL; visual mesh filename=package://stretch_description/meshes/link_aruco_shoulder.STL
- link link_aruco_top_wrist: geometry collision mesh filename=package://stretch_description/meshes/link_aruco_top_wrist.S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; visual mesh filename=package://stretch_description/meshes/link_aruco_top_wrist.S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
- link link_gripper_finger_left: geometry collision mesh filename=package://stretch_description/meshes/link_gripper_finger_le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; visual mesh filename=package://stretch_description/meshes/link_gripper_finger_le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
- link link_gripper_finger_right: geometry collision mesh filename=package://stretch_description/meshes/link_gripper_finger_ri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; visual mesh filename=package://stretch_description/meshes/link_gripper_finger_ri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
- link link_gripper_fingertip_left: geometry collision mesh filename=package://stretch_description/meshes/link_gripper_fingertip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; visual mesh filename=package://stretch_description/meshes/link_gripper_fingertip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
- link link_gripper_fingertip_right: geometry collision mesh filename=package://stretch_description/meshes/link_gripper_fingertip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; visual mesh filename=package://stretch_description/meshes/link_gripper_fingertip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
- link link_head: geometry collision mesh filename=package://stretch_description/meshes/link_head.STL; visual mesh filename=package://stretch_description/meshes/link_head.STL
- link link_head_pan: geometry collision mesh filename=package://stretch_description/meshes/link_head_pan.STL; visual mesh filename=package://stretch_description/meshes/link_head_pan.STL
- link link_head_tilt: geometry collision mesh filename=package://stretch_description/meshes/link_head_tilt.STL; visual mesh filename=package://stretch_description/meshes/link_head_tilt.STL
- link link_left_wheel: geometry collision mesh filename=package://stretch_description/meshes/link_left_wheel.STL; visual mesh filename=package://stretch_description/meshes/link_left_wheel.STL
- link link_lift: geometry collision mesh filename=package://stretch_description/meshes/link_lift.STL; visual mesh filename=package://stretch_description/meshes/link_lift.STL
- link link_mast: geometry collision mesh filename=package://stretch_description/meshes/link_mast.STL; visual mesh filename=package://stretch_description/meshes/link_mast.STL
- link link_right_wheel: geometry collision mesh filename=package://stretch_description/meshes/link_right_wheel.STL; visual mesh filename=package://stretch_description/meshes/link_right_wheel.STL
- link link_straight_gripper: geometry collision mesh filename=package://stretch_description/meshes/link_straight_gripper.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; visual mesh filename=package://stretch_description/meshes/link_straight_gripper.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
- link link_wrist_pitch: geometry collision mesh filename=package://stretch_description/meshes/link_wrist_pitch.STL; visual mesh filename=package://stretch_description/meshes/link_wrist_pitch.STL
- link link_wrist_roll: geometry collision mesh filename=package://stretch_description/meshes/link_wrist_roll.STL; visual mesh filename=package://stretch_description/meshes/link_wrist_roll.STL
- link link_wrist_yaw: geometry collision mesh filename=package://stretch_description/meshes/link_wrist_yaw.STL; visual mesh filename=package://stretch_description/meshes/link_wrist_yaw.STL
- link link_wrist_yaw_bottom: geometry collision mesh filename=package://stretch_description/meshes/link_wrist_yaw_bottom.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; visual mesh filename=package://stretch_description/meshes/link_wrist_yaw_bottom.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
- link respeaker_base: geometry collision mesh filename=package://stretch_description/meshes/respeaker_base.STL; visual mesh filename=package://stretch_description/meshes/respeaker_base.STL
